File: esp32p4_lte_cam.kicad_pcb (KiCad board)
At the start: 4 copper layers, 0 parts

Commit message: Phase 3: board setup
- Netlist -> PCB sync script (keeps placement, schematic links, LCSC/MPN fields)
- 75x70 mm outline, 4x M2.5 GND holes, JLC04161H-7628 stackup, L2 GND plane
- Net classes by pattern (Power, HighCurrent, RF 50R CPWG, USB 90R, MIPI 100R),
  JLC-checked rules and custom DRC rules; impedance calculator script
- Library fixes: peg holes -> NPTH, PIR courtyard, Espressif supply pin types
- Short sheet names so local nets read /power/..., /mcu/...
- DRC 0 violations; 231 footprints staged for placement

Co-Authored-By: Claude Opus 5.5 <noreply@anthropic.com>
Parts:
- added C201: 1u 25V, Capacitor_SMD:C_0603_1608Metric, F.Cu at (112.5, 1.75)
- added C202: 10u 25V, Capacitor_SMD:C_0805_2012Metric, F.Cu at (112.7, 5.51)
- added C203: 4.7u 10V, Capacitor_SMD:C_0603_1608Metric, F.Cu at (112.5, 9.27)
- added C204: 47n 16V, Capacitor_SMD:C_0402_1005Metric, F.Cu at (111.9, 12.5)
- added C205: 10u 10V, Capacitor_SMD:C_0805_2012Metric, F.Cu at (112.7, 16.0)
- added C206: 10u 10V, Capacitor_SMD:C_0805_2012Metric, F.Cu at (112.7, 20.0)
- added C207: 10u 10V, Capacitor_SMD:C_0805_2012Metric, F.Cu at (112.7, 24.0)
- added C208: 100n, Capacitor_SMD:C_0402_1005Metric, F.Cu at (111.9, 27.5)
- added C209: 22u 10V, Capacitor_SMD:C_0805_2012Metric, F.Cu at (112.7, 31.0)
- added C210: 10p, Capacitor_SMD:C_0402_1005Metric, F.Cu at (111.9, 34.5)
- added C211: 22u 10V, Capacitor_SMD:C_0805_2012Metric, F.Cu at (112.7, 38.0)
- added C212: 22u 10V, Capacitor_SMD:C_0805_2012Metric, F.Cu at (112.7, 42.0)
- added C213: 100n, Capacitor_SMD:C_0402_1005Metric, F.Cu at (111.9, 45.5)
- added C214: 1u, Capacitor_SMD:C_0402_1005Metric, F.Cu at (111.9, 48.5)
- added C215: 1u, Capacitor_SMD:C_0402_1005Metric, F.Cu at (111.9, 51.4)
- added C301: 100n, Capacitor_SMD:C_0402_1005Metric, F.Cu at (125.2, 57.6)
- added C302: 100n, Capacitor_SMD:C_0402_1005Metric, F.Cu at (125.2, 60.6)
- added C303: 100n, Capacitor_SMD:C_0402_1005Metric, F.Cu at (125.2, 63.6)
- added C304: 100n, Capacitor_SMD:C_0402_1005Metric, F.Cu at (125.2, 66.5)
- added C305: 100n, Capacitor_SMD:C_0402_1005Metric, F.Cu at (125.2, 69.5)
- added C306: 100n, Capacitor_SMD:C_0402_1005Metric, F.Cu at (125.2, 72.5)
- added C307: 100n, Capacitor_SMD:C_0402_1005Metric, F.Cu at (125.2, 75.5)
- added C308: 10u 10V, Capacitor_SMD:C_0603_1608Metric, F.Cu at (125.8, 78.7)
- added C309: 10u 10V, Capacitor_SMD:C_0603_1608Metric, F.Cu at (125.8, 82.2)
- added C310: 10u 10V, Capacitor_SMD:C_0603_1608Metric, F.Cu at (125.8, 85.7)
- added C311: 100n, Capacitor_SMD:C_0402_1005Metric, F.Cu at (125.2, 89.0)
- added C312: 100n, Capacitor_SMD:C_0402_1005Metric, F.Cu at (125.2, 91.9)
- added C313: 100n, Capacitor_SMD:C_0402_1005Metric, F.Cu at (125.2, 94.9)
- added C314: 100n, Capacitor_SMD:C_0402_1005Metric, F.Cu at (125.2, 97.9)
- added C315: 10u 10V, Capacitor_SMD:C_0603_1608Metric, F.Cu at (125.8, 101.1)
- added C316: 1u, Capacitor_SMD:C_0402_1005Metric, F.Cu at (125.2, 104.3)
- added C317: 100n, Capacitor_SMD:C_0402_1005Metric, F.Cu at (125.2, 107.3)
- added C318: 1u, Capacitor_SMD:C_0402_1005Metric, F.Cu at (125.2, 110.3)
- added C319: 100n, Capacitor_SMD:C_0402_1005Metric, F.Cu at (125.2, 113.3)
- added C320: 100n, Capacitor_SMD:C_0402_1005Metric, F.Cu at (125.2, 116.2)
- added C321: 1u, Capacitor_SMD:C_0402_1005Metric, F.Cu at (132.5, 1.48)
- added C322: 1u, Capacitor_SMD:C_0402_1005Metric, F.Cu at (132.5, 4.46)
- added C323: 100n, Capacitor_SMD:C_0402_1005Metric, F.Cu at (132.5, 7.42)
- added C324: 10n, Capacitor_SMD:C_0402_1005Metric, F.Cu at (132.5, 10.4)
- added C325: 1u, Capacitor_SMD:C_0402_1005Metric, F.Cu at (132.5, 13.4)
- added C326: 100n, Capacitor_SMD:C_0402_1005Metric, F.Cu at (132.5, 16.3)
- added C327: 1u, Capacitor_SMD:C_0402_1005Metric, F.Cu at (132.5, 19.3)
- added C328: 4.7u 10V, Capacitor_SMD:C_0603_1608Metric, F.Cu at (133.1, 22.5)
- added C329: 22p, Capacitor_SMD:C_0402_1005Metric, F.Cu at (132.5, 25.8)
- added C330: 22u 10V, Capacitor_SMD:C_0805_2012Metric, F.Cu at (133.3, 29.3)
- added C331: 100n, Capacitor_SMD:C_0402_1005Metric, F.Cu at (132.5, 32.8)
- added C332: 22p, Capacitor_SMD:C_0402_1005Metric, F.Cu at (132.5, 35.7)
- added C333: 22p, Capacitor_SMD:C_0402_1005Metric, F.Cu at (132.5, 38.7)
- added C334: 18p, Capacitor_SMD:C_0402_1005Metric, F.Cu at (132.5, 41.7)
- added C335: 18p, Capacitor_SMD:C_0402_1005Metric, F.Cu at (132.5, 44.6)
- added C336: 100n, Capacitor_SMD:C_0402_1005Metric, F.Cu at (132.5, 47.6)
- added C401: 10u 10V, Capacitor_SMD:C_0603_1608Metric, F.Cu at (139.0, 82.6)
- added C402: 100n, Capacitor_SMD:C_0402_1005Metric, F.Cu at (138.4, 85.8)
- added C403: 1u, Capacitor_SMD:C_0402_1005Metric, F.Cu at (138.4, 88.8)
- added C501: 220u 6.3V, Capacitor_Tantalum_SMD:CP_EIA-3528-21_Kemet-B, F.Cu at (154.0, 42.0)
- added C502: 220u 6.3V, Capacitor_Tantalum_SMD:CP_EIA-3528-21_Kemet-B, F.Cu at (154.0, 47.4)
- added C503: 10u 10V, Capacitor_SMD:C_0603_1608Metric, F.Cu at (153.0, 51.8)
- added C504: 100n, Capacitor_SMD:C_0402_1005Metric, F.Cu at (152.5, 55.1)
- added C505: 33p, Capacitor_SMD:C_0402_1005Metric, F.Cu at (152.5, 58.0)
- added C506: 10p, Capacitor_SMD:C_0402_1005Metric, F.Cu at (152.5, 61.0)
- added C507: 1u, Capacitor_SMD:C_0402_1005Metric, F.Cu at (152.5, 64.0)
- added C508: 10u 10V, Capacitor_SMD:C_0805_2012Metric, F.Cu at (153.3, 67.5)
- added C509: 1n 25V, Capacitor_SMD:C_0402_1005Metric, F.Cu at (152.5, 71.0)
- added C510: 100n 16V, Capacitor_SMD:C_0402_1005Metric, F.Cu at (152.5, 73.9)
- added C511: 100n, Capacitor_SMD:C_0402_1005Metric, F.Cu at (152.5, 76.9)
- added C512: 100n, Capacitor_SMD:C_0402_1005Metric, F.Cu at (152.5, 79.9)
- added C513: 33p, Capacitor_SMD:C_0402_1005Metric, F.Cu at (152.5, 82.8)
- added C514: 33p, Capacitor_SMD:C_0402_1005Metric, F.Cu at (152.5, 85.8)
- added C515: 33p, Capacitor_SMD:C_0402_1005Metric, F.Cu at (152.5, 88.8)
- added C516: 100n, Capacitor_SMD:C_0402_1005Metric, F.Cu at (152.5, 91.7)
- added C517: DNP, Capacitor_SMD:C_0402_1005Metric, F.Cu at (152.5, 94.7)
- added C518: DNP, Capacitor_SMD:C_0402_1005Metric, F.Cu at (152.5, 97.7)
- added C519: DNP, Capacitor_SMD:C_0402_1005Metric, F.Cu at (152.5, 100.7)
- added C520: DNP, Capacitor_SMD:C_0402_1005Metric, F.Cu at (152.5, 103.6)
- added C521: DNP, Capacitor_SMD:C_0402_1005Metric, F.Cu at (152.5, 106.6)
- added C522: DNP, Capacitor_SMD:C_0402_1005Metric, F.Cu at (152.5, 109.6)
- added C601: 10u 10V, Capacitor_SMD:C_0603_1608Metric, F.Cu at (184.5, 50.9)
- added C602: 100n, Capacitor_SMD:C_0402_1005Metric, F.Cu at (183.9, 54.1)
- added C603: 1n 25V, Capacitor_SMD:C_0402_1005Metric, F.Cu at (183.9, 57.1)
- added C604: 1u, Capacitor_SMD:C_0402_1005Metric, F.Cu at (183.9, 60.0)
- added C605: 10u 10V, Capacitor_SMD:C_0805_2012Metric, F.Cu at (184.7, 63.5)
- added C606: 4.7u 25V, Capacitor_SMD:C_0805_2012Metric, F.Cu at (184.7, 67.5)
- added C607: 10u 10V, Capacitor_SMD:C_0805_2012Metric, F.Cu at (184.7, 71.6)
- added C608: 100n 16V, Capacitor_SMD:C_0402_1005Metric, F.Cu at (183.9, 75.0)
- added C609: 100n, Capacitor_SMD:C_0402_1005Metric, F.Cu at (183.9, 78.0)
- added C610: 4.7u 10V, Capacitor_SMD:C_0603_1608Metric, F.Cu at (184.5, 81.3)
- added C611: 100n, Capacitor_SMD:C_0402_1005Metric, F.Cu at (183.9, 84.5)
- added C701: DNP, Capacitor_SMD:C_0402_1005Metric, F.Cu at (218.9, 78.6)
- added C702: 10u 10V, Capacitor_SMD:C_0603_1608Metric, F.Cu at (219.4, 81.9)
- added C703: 100n, Capacitor_SMD:C_0402_1005Metric, F.Cu at (218.9, 85.1)
- added C704: 1n 25V, Capacitor_SMD:C_0402_1005Metric, F.Cu at (218.9, 88.1)
- added C705: 1u, Capacitor_SMD:C_0402_1005Metric, F.Cu at (218.9, 91.1)
- added D201: SMF5.0A (TVS), Diode_SMD:D_SOD-123F, F.Cu at (113.2, 55.1)
- added D601: B5819W, Diode_SMD:D_SOD-123, F.Cu at (185.4, 88.2)
- added D602: IR 850nm, lcsc:LED-SMD_3P-L3.8-W3.8_M3838E1IRS1G09, F.Cu at (185.3, 93.3)
- added D603: IR 850nm, lcsc:LED-SMD_3P-L3.8-W3.8_M3838E1IRS1G09, F.Cu at (185.3, 99.2)
- added D604: IR 850nm, lcsc:LED-SMD_3P-L3.8-W3.8_M3838E1IRS1G09, F.Cu at (185.3, 105.1)
- added D605: IR 850nm, lcsc:LED-SMD_3P-L3.8-W3.8_M3838E1IRS1G09, F.Cu at (185.3, 111.0)
- added H1: M2.5, MountingHole:MountingHole_2.7mm_M2.5_Pad_Via, F.Cu at (3.50, 9.50)
- added H2: M2.5, MountingHole:MountingHole_2.7mm_M2.5_Pad_Via, F.Cu at (71.5, 9.50)
- added H3: M2.5, MountingHole:MountingHole_2.7mm_M2.5_Pad_Via, F.Cu at (3.50, 66.5)
- added H4: M2.5, MountingHole:MountingHole_2.7mm_M2.5_Pad_Via, F.Cu at (71.5, 66.5)
- added J1: USB-C (bottom edge), Connector_USB:USB_C_Receptacle_HRO_TYPE-C-31-M-12, F.Cu at (116.3, 63.0)
- added J2: CAM FPC 22P 0.5mm, lcsc:CONN-SMD_05B20L22P, F.Cu at (226.4, 3.85)
- added J3: microSD, lcsc:TF-SMD_TF-01A, F.Cu at (226.3, 101.4)
- added J4: Nano-SIM, lcsc:SIM-SMD_NANO-SIM-7P-H1.37, F.Cu at (174.1, 8.62)
- added J5: U.FL MAIN, lcsc:RF-SMD_FRF05002-JSS103M, F.Cu at (169.2, 20.1)
- added J6: U.FL AUX, lcsc:RF-SMD_FRF05002-JSS103M, F.Cu at (169.2, 25.9)
- added J7: U.FL GNSS, lcsc:RF-SMD_FRF05002-JSS103M, F.Cu at (169.2, 31.6)
- added J8: BATT (+ / NTC / -), Connector_JST:JST_PH_S3B-PH-SM4-TB_1x03-1MP_P2.00mm_Horizontal, F.Cu at (116.6, 74.9)
- added J9: IR-CUT, Connector_JST:JST_SH_SM02B-SRSS-TB_1x02-1MP_P1.00mm_Horizontal, F.Cu at (220.9, 12.0)
- added L201: 2.2uH, lcsc:IND-SMD_L5.0-W5.0_SMNR5030, F.Cu at (114.0, 84.7)
- added L202: 1uH, Inductor_SMD:L_1008_2520Metric, F.Cu at (113.0, 90.8)
- added L301: 2.2uH, Inductor_SMD:L_1008_2520Metric, F.Cu at (133.5, 51.5)
- added L501: 47nH, Inductor_SMD:L_0402_1005Metric, F.Cu at (168.2, 36.0)
- added L601: 10uH, lcsc:IND-SMD_L4.0-W4.0, F.Cu at (220.3, 19.5)
- added Q201: FS8205A, lcsc:SOT-23-6_L2.9-W1.6-P0.95-LS2.8-BR, F.Cu at (112.9, 96.0)
- added Q501: 2N7002, Package_TO_SOT_SMD:SOT-23, F.Cu at (169.2, 40.2)
- added Q502: 2N7002, Package_TO_SOT_SMD:SOT-23, F.Cu at (169.2, 45.7)
- added R201: 5.1k, Resistor_SMD:R_0402_1005Metric, F.Cu at (112.0, 100.2)
- added R202: 5.1k, Resistor_SMD:R_0402_1005Metric, F.Cu at (112.0, 103.2)
- added R203: 0, Resistor_SMD:R_0402_1005Metric, F.Cu at (112.0, 106.2)
- added R204: 0, Resistor_SMD:R_0402_1005Metric, F.Cu at (112.0, 109.2)
- added R205: 120, Resistor_SMD:R_0402_1005Metric, F.Cu at (112.0, 112.2)
- added R206: 5.23k, Resistor_SMD:R_0402_1005Metric, F.Cu at (112.0, 115.2)
- added R207: 30.1k, Resistor_SMD:R_0402_1005Metric, F.Cu at (112.0, 118.2)
- added R208: 10k, Resistor_SMD:R_0402_1005Metric, F.Cu at (125.2, 1.50)
- added R209: 10k, Resistor_SMD:R_0402_1005Metric, F.Cu at (125.2, 4.49)
- added R210: 10k, Resistor_SMD:R_0402_1005Metric, F.Cu at (125.2, 7.47)
- added R211: 100, Resistor_SMD:R_0402_1005Metric, F.Cu at (125.2, 10.5)
- added R212: 1k, Resistor_SMD:R_0402_1005Metric, F.Cu at (125.2, 13.5)
- added R213: 560k, Resistor_SMD:R_0402_1005Metric, F.Cu at (125.2, 16.4)
- added R214: 100k, Resistor_SMD:R_0402_1005Metric, F.Cu at (125.2, 19.4)
- added R301: 4.02k, Resistor_SMD:R_0402_1005Metric, F.Cu at (132.5, 55.3)
- added R302: 499k, Resistor_SMD:R_0402_1005Metric, F.Cu at (132.5, 58.3)
- added R303: 499k, Resistor_SMD:R_0402_1005Metric, F.Cu at (132.5, 61.3)
- added R304: 0, Resistor_SMD:R_0402_1005Metric, F.Cu at (132.5, 64.3)
- added R305: 0, Resistor_SMD:R_0402_1005Metric, F.Cu at (132.5, 67.3)
- added R306: 0, Resistor_SMD:R_0402_1005Metric, F.Cu at (132.5, 70.3)
- added R307: 0, Resistor_SMD:R_0402_1005Metric, F.Cu at (132.5, 73.3)
- added R308: 0, Resistor_SMD:R_0402_1005Metric, F.Cu at (132.5, 76.3)
- added R309: 0, Resistor_SMD:R_0402_1005Metric, F.Cu at (132.5, 79.3)
- added R310: 10k, Resistor_SMD:R_0402_1005Metric, F.Cu at (132.5, 82.3)
- added R311: 1k, Resistor_SMD:R_0402_1005Metric, F.Cu at (132.5, 85.2)
- added R312: 10k, Resistor_SMD:R_0402_1005Metric, F.Cu at (132.5, 88.2)
- added R313: 10k, Resistor_SMD:R_0402_1005Metric, F.Cu at (132.5, 91.2)
- added R314: 22, Resistor_SMD:R_0402_1005Metric, F.Cu at (132.5, 94.2)
- added R315: 22, Resistor_SMD:R_0402_1005Metric, F.Cu at (132.5, 97.2)
- added R316: 0, Resistor_SMD:R_0402_1005Metric, F.Cu at (132.5, 100.2)
- added R317: 0, Resistor_SMD:R_0402_1005Metric, F.Cu at (132.5, 103.2)
- added R318: 0, Resistor_SMD:R_0402_1005Metric, F.Cu at (132.5, 106.2)
- added R319: 0, Resistor_SMD:R_0402_1005Metric, F.Cu at (132.5, 109.2)
- added R320: 0, Resistor_SMD:R_0402_1005Metric, F.Cu at (132.5, 112.2)
- added R321: 0, Resistor_SMD:R_0402_1005Metric, F.Cu at (132.5, 115.1)
- added R401: 10k, Resistor_SMD:R_0402_1005Metric, F.Cu at (138.5, 91.8)
- added R402: 10k, Resistor_SMD:R_0402_1005Metric, F.Cu at (138.5, 94.8)
- added R403: 10k, Resistor_SMD:R_0402_1005Metric, F.Cu at (138.5, 97.8)
- added R404: 10k, Resistor_SMD:R_0402_1005Metric, F.Cu at (138.5, 100.7)
- added R405: 10k, Resistor_SMD:R_0402_1005Metric, F.Cu at (138.5, 103.7)
- added R406: 10k, Resistor_SMD:R_0402_1005Metric, F.Cu at (138.5, 106.7)
- added R407: 10k, Resistor_SMD:R_0402_1005Metric, F.Cu at (138.5, 109.7)
- added R408: 10k, Resistor_SMD:R_0402_1005Metric, F.Cu at (138.5, 112.7)
- added R501: 100k, Resistor_SMD:R_0402_1005Metric, F.Cu at (168.2, 49.9)
- added R502: 100k, Resistor_SMD:R_0402_1005Metric, F.Cu at (168.2, 52.9)
- added R503: 100k, Resistor_SMD:R_0402_1005Metric, F.Cu at (168.2, 55.9)
- added R504: 100k, Resistor_SMD:R_0402_1005Metric, F.Cu at (168.2, 58.9)
- added R505: 22, Resistor_SMD:R_0402_1005Metric, F.Cu at (168.2, 61.9)
- added R506: 22, Resistor_SMD:R_0402_1005Metric, F.Cu at (168.2, 64.9)
- added R507: 22, Resistor_SMD:R_0402_1005Metric, F.Cu at (168.2, 67.9)
- added R508: 10k, Resistor_SMD:R_0402_1005Metric, F.Cu at (168.2, 70.8)
- added R509: 0, Resistor_SMD:R_0402_1005Metric, F.Cu at (168.2, 73.8)
- added R510: 0, Resistor_SMD:R_0402_1005Metric, F.Cu at (168.2, 76.8)
- added R511: 0, Resistor_SMD:R_0402_1005Metric, F.Cu at (168.2, 79.8)
- added R512: 10, Resistor_SMD:R_0402_1005Metric, F.Cu at (168.2, 82.8)
- added R601: 2.2k, Resistor_SMD:R_0402_1005Metric, F.Cu at (218.9, 24.1)
- added R602: 2.2k, Resistor_SMD:R_0402_1005Metric, F.Cu at (218.9, 27.1)
- added R603: 10k, Resistor_SMD:R_0402_1005Metric, F.Cu at (218.9, 30.1)
- added R604: 10k, Resistor_SMD:R_0402_1005Metric, F.Cu at (218.9, 33.1)
- added R605: 100k, Resistor_SMD:R_0402_1005Metric, F.Cu at (218.9, 36.1)
- added R606: 0.68, Resistor_SMD:R_0805_2012Metric, F.Cu at (219.7, 39.6)
- added R607: 100k, Resistor_SMD:R_0402_1005Metric, F.Cu at (218.9, 43.0)
- added R608: 100k, Resistor_SMD:R_0402_1005Metric, F.Cu at (218.9, 46.0)
- added R609: 100, Resistor_SMD:R_0402_1005Metric, F.Cu at (218.9, 49.0)
- added R701: 22, Resistor_SMD:R_0402_1005Metric, F.Cu at (218.9, 111.7)
- added R702: 10k, Resistor_SMD:R_0402_1005Metric, F.Cu at (218.9, 114.7)
- added R703: 10k, Resistor_SMD:R_0402_1005Metric, F.Cu at (218.9, 117.6)
- added R704: 10k, Resistor_SMD:R_0402_1005Metric, F.Cu at (237.8, 1.50)
- added R705: 10k, Resistor_SMD:R_0402_1005Metric, F.Cu at (237.8, 4.49)
- added R706: 10k, Resistor_SMD:R_0402_1005Metric, F.Cu at (237.8, 7.47)
- added R707: 10k, Resistor_SMD:R_0402_1005Metric, F.Cu at (237.8, 10.5)
- added R708: 100k, Resistor_SMD:R_0402_1005Metric, F.Cu at (237.8, 13.5)
- added RT201: 10k B3435 (DNP), Resistor_SMD:R_0603_1608Metric, F.Cu at (125.8, 22.7)
- added SW301: RESET, lcsc:SW-SMD_L4.0-W2.9-P4.15-EH, F.Cu at (140.3, 2.58)
- added SW302: BOOT, lcsc:SW-SMD_L4.0-W2.9-P4.15-EH, F.Cu at (140.3, 7.72)
- added TP201: CHG_QON, TestPoint:TestPoint_Pad_D1.0mm, F.Cu at (125.3, 26.5)
- added TP301: UART0_TX, TestPoint:TestPoint_Pad_D1.0mm, F.Cu at (138.5, 12.3)
- added TP302: UART0_RX, TestPoint:TestPoint_Pad_D1.0mm, F.Cu at (138.5, 16.4)
- added TP303: BOOT, TestPoint:TestPoint_Pad_D1.0mm, F.Cu at (138.5, 20.4)
- added TP304: CHIP_PU, TestPoint:TestPoint_Pad_D1.0mm, F.Cu at (138.5, 24.5)
- added TP305: TP_GPIO12, TestPoint:TestPoint_Pad_D1.0mm, F.Cu at (138.5, 28.5)
- added TP306: TP_GPIO13, TestPoint:TestPoint_Pad_D1.0mm, F.Cu at (138.5, 32.6)
- added TP307: TP_GPIO33, TestPoint:TestPoint_Pad_D1.0mm, F.Cu at (138.5, 36.6)
- added TP401: C6_TXD0, TestPoint:TestPoint_Pad_D1.0mm, F.Cu at (138.5, 116.2)
- added TP402: C6_RXD0, TestPoint:TestPoint_Pad_D1.0mm, F.Cu at (152.6, 2.02)
- added TP403: C6_EN, TestPoint:TestPoint_Pad_D1.0mm, F.Cu at (152.6, 6.07)
- added TP404: C6_BOOT, TestPoint:TestPoint_Pad_D1.0mm, F.Cu at (152.6, 10.1)
- added TP405: C6_USB_DN, TestPoint:TestPoint_Pad_D1.0mm, F.Cu at (152.6, 14.2)
- added TP406: C6_USB_DP, TestPoint:TestPoint_Pad_D1.0mm, F.Cu at (152.6, 18.2)
- added TP501: MDM_1V8, TestPoint:TestPoint_Pad_D1.0mm, F.Cu at (168.3, 86.3)
- added TP502: MDM_USB_VBUS, TestPoint:TestPoint_Pad_D1.0mm, F.Cu at (168.3, 90.4)
- added TP503: MDM_USB_DP, TestPoint:TestPoint_Pad_D1.0mm, F.Cu at (168.3, 94.4)
- added TP504: MDM_USB_DN, TestPoint:TestPoint_Pad_D1.0mm, F.Cu at (168.3, 98.5)
- added TP505: MDM_DBG_TXD, TestPoint:TestPoint_Pad_D1.0mm, F.Cu at (168.3, 102.5)
- added TP506: MDM_DBG_RXD, TestPoint:TestPoint_Pad_D1.0mm, F.Cu at (168.3, 106.6)
- added U1: ESP32-P4NRW32X, espressif:ESP32-P4, F.Cu at (143.5, 45.3)
- added U10: TPS22918, lcsc:SOT-23-6_L2.9-W1.6-P0.95-LS2.8-BR, F.Cu at (219.8, 53.3)
- added U11: TPS22918, lcsc:SOT-23-6_L2.9-W1.6-P0.95-LS2.8-BR, F.Cu at (238.7, 17.7)
- added U12: TPS61169, lcsc:SC-70-5_L2.1-W1.3-P0.65-LS2.1-BR, F.Cu at (219.5, 58.5)
- added U13: DRV8837, Package_SON:Texas_DSG0008A_WSON-8-1EP_2x2mm_P0.5mm_EP0.9x1.6mm, F.Cu at (219.5, 63.2)
- added U14: DW01A, Package_TO_SOT_SMD:SOT-23-6, F.Cu at (126.3, 48.1)
- added U15: TPS3839G33 (3.08V), Package_TO_SOT_SMD:SOT-23, F.Cu at (139.5, 68.2)
- added U16: SN74LVC1T45, Package_TO_SOT_SMD:SOT-23-6, F.Cu at (185.0, 41.0)
- added U17: TPD4E05U06, Package_SON:USON-10_2.5x1.0mm_P0.5mm, F.Cu at (125.2, 53.5)
- added U18: TPD4E05U06, Package_SON:USON-10_2.5x1.0mm_P0.5mm, F.Cu at (183.9, 46.5)
- added U19: XYC-PIR223D-S0, lcsc:TO-5-3_L8.2-W8.2, F.Cu at (222.7, 71.4)
- added U2: W25Q128JVSIQ, Package_SO:SOIC-8_5.3x5.3mm_P1.27mm, F.Cu at (142.2, 55.9)
- added U3: ESP32-C6-MINI-1, espressif:ESP32-C6-MINI-1, F.Cu at (158.4, 29.8)
- added U4: SIM7600G-H, lcsc:COMM-SMD_135P-L30.0-W30.0_SIM7600G, F.Cu at (199.4, 16.9)
- added U5: BQ25895RTWR, Package_DFN_QFN:Texas_RTW_WQFN-24-1EP_4x4mm_P0.5mm_EP2.7x2.7mm_ThermalVias, F.Cu at (126.9, 32.1)
- added U6: TPS631000, lcsc:SOT-583-8_L2.1-W1.2-P0.50-LS1.6-BL, F.Cu at (125.6, 37.8)
- added U7: TLV62569, Package_TO_SOT_SMD:SOT-23-5, F.Cu at (139.6, 62.7)
- added U8: TPS7A0218, lcsc:SOT-23-5_L3.0-W1.7-P0.95-LS2.8-BL, F.Cu at (126.0, 42.5)
- added U9: TPS22965, lcsc:UDFN-8_L2.0-W2.0-P0.50-TL-EP, F.Cu at (184.4, 36.1)
- added Y1: 40MHz 10ppm, Crystal:Crystal_SMD_3225-4Pin_3.2x2.5mm, F.Cu at (139.6, 73.7)
- added Y2: 32.768kHz, Crystal:Crystal_SMD_3215-2Pin_3.2x1.5mm, F.Cu at (139.5, 78.7)
Routing:
- added copper zone on In1.Cu, net GND
Other:
- board outline added: 75 x 70 mm

Commit message: Phase 4: placement (Review 3)
- Scripted placement: anchors per floor plan + pin-attraction satellites
  (switch-node parts hug their regulator, decaps spread over owner pins);
  pad-aware collision boxes; optional --p4-decaps-bottom variant
- P4 rotated 180 for a straight 11 mm CSI path; card slots moved to edges
  (nano-SIM bottom, microSD west); C6 module NE corner, antenna on edge
- Fiducials, SIM7600 top-layer no-track rule area, bottom silk legends
- Silkscreen tidy pipeline (KRT beautify_labels + DRC-driven hiding,
  clear-spot seating for key designators)
- Library: imported silk trimmed off pads, P4 3D model, C6 model path
- DRC 0 violations; renders, assembly drawing, metrics, review doc

Co-Authored-By: Claude Opus 5.5 <noreply@anthropic.com>
Parts:
- added FID1: Fiducial, Fiducial:Fiducial_1mm_Mask2mm, F.Cu at (8.50, 10.8)
- added FID2: Fiducial, Fiducial:Fiducial_1mm_Mask2mm, F.Cu at (59.3, 3.53)
- added FID3: Fiducial, Fiducial:Fiducial_1mm_Mask2mm, F.Cu at (38.5, 66.5)
- moved J3 230.8 mm to (9.90, 21.0), turned to -90 degrees
- moved R703 221.2 mm to (20.7, 19.4)
- moved R702 218.7 mm to (21.2, 21.1), turned to 90 degrees
- moved R704 218.1 mm to (20.2, 18.1)
- moved R706 217.3 mm to (21.1, 22.9)
- moved R705 215.3 mm to (23.1, 20.6)
- moved R701 215.2 mm to (23.2, 21.9)
- moved U11 213.7 mm to (25.0, 18.4)
- moved C703 211.5 mm to (18.2, 18.2), turned to 90 degrees
- moved R707 211.4 mm to (26.6, 21.3), turned to 90 degrees
- moved U19 211.4 mm to (21.5, 6.60)
- moved C702 210.9 mm to (17.8, 20.4)
- moved C701 210.8 mm to (16.9, 18.2), turned to 90 degrees
- moved R609 209.5 mm to (14.0, 5.60), turned to 90 degrees
- moved C704 209.2 mm to (22.2, 16.8), turned to 90 degrees
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Other:
- board text added: "ANT DIV"
- board text added: "ANT MAIN"
- board text added: "BATT +/NTC/-"
- board text added: "CAMERA"
- board text added: "ESP32-P4 LTE CAMERA"
- board text added: "GNSS"
- board text added: "H. Jimenez | 4L JLC04161H-7628"
- board text added: "IR-CUT"
- board text added: "NANO-SIM"
- board text added: "USB-C 5V"
- board text added: "Wi-Fi 6 / BLE"
- board text added: "microSD"
- board text added: "rev A - 2026-10"

Commit message: Phase 5 prep: bottom-side P4 decoupling, plane split, MIPI hand route
- place.py: P4 decaps on B.Cu by default, U9 moved south-west of modem
- planes.py: GND L1/L2/L4, hand split L3 (VBAT_LTE / SYS / 3V3)
- route_mipi.py: coupled 100R CSI pairs, clock crossover via B.Cu
- viewroute.py: region render of pads/tracks/vias
- board_setup.py: MIPI intra-pair skew 0.3 mm

Co-Authored-By: Claude Opus 5.5 <noreply@anthropic.com>
Parts:
- C301, C302, C303, C304, C305, C306, C307, C311, C312, C313, C314, C316, C317, C318, C319, C320, C321, C322, C323, C324, C325, C326, C327, C331: moved to B.Cu
- moved C508 45.3 mm to (38.8, 66.2), turned to 90 degrees
- moved C509 44.4 mm to (44.0, 68.0)
- moved U9 44.2 mm to (41.5, 67.4)
- moved R501 28.9 mm to (36.6, 47.3)
- moved TP405 19.0 mm to (59.4, 11.8)
- moved C521 18.5 mm to (52.2, 31.1)
- moved TP404 16.7 mm to (58.6, 28.3)
- moved TP306 12.7 mm to (55.6, 15.1)
- moved C308 10.3 mm to (39.9, 28.5)
- moved C202 9.80 mm to (14.2, 38.1)
- moved TP406 9.42 mm to (61.8, 11.8)
- moved R310 8.86 mm to (31.3, 20.4), turned to 90 degrees
- moved FID3 8.42 mm to (46.8, 65.8)
- moved C333 8.14 mm to (46.0, 21.8)
- moved C326 8.00 mm to (41.5, 27.4)
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
Commit message: Phase 5: USB hookup (P4 escape, J1/ESD/CC hand route, BC1.2 taps)
- place.py: anchor R314/R315 on B.Cu beside the P4 USB corner, keep-clear corridors
- route_usb.py: P4 USB escape to the 22R pair; J1 -> B.Cu coupled pair
  (0.22/0.13) under U17 to R314/R315 with short ESD taps; CC1/CC2 to
  U17 and the 5.1k pull-downs via B.Cu links under the J1 pad row
- CHG_DP/CHG_DN and the R203/R204 BC1.2 taps autorouted (KRT route.py)
- DRC: no clearance violations; remaining items are unrouted nets

Co-Authored-By: Claude Opus 5.5 <noreply@anthropic.com>
Parts:
- R314, R315: moved to B.Cu
- moved R315 37.1 mm to (29.9, 13.4), turned to 180 degrees
- moved R314 34.8 mm to (29.9, 14.6), turned to 180 degrees
- moved R603 10.8 mm to (45.0, 9.15)
- moved R203 10.4 mm to (21.3, 43.9), turned to 0 degrees
- moved C202 10.1 mm to (19.6, 46.6), turned to 90 degrees
- moved C209 7.91 mm to (16.0, 51.6), turned to 0 degrees
- moved R607 7.30 mm to (46.2, 16.4)
- moved C204 6.66 mm to (13.1, 43.5), turned to 90 degrees
- moved C215 6.64 mm to (15.9, 53.4), turned to 0 degrees
- moved R608 5.19 mm to (48.5, 11.6)
- moved TP303 4.34 mm to (14.7, 38.2)
- moved R204 3.70 mm to (13.5, 51.5)
- moved R309 3.44 mm to (51.0, 11.4), turned to 90 degrees
- moved C207 3.01 mm to (19.7, 52.0)
- moved R308 2.59 mm to (48.0, 9.45), turned to 0 degrees
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Routing:
- net USB_DN: track 0.00 -> 63.8 mm, vias 0 -> 3
- net USB_DP: track 0.00 -> 62.6 mm, vias 0 -> 3
- net /power/USB_CC2: track 0.00 -> 13.9 mm, vias 0 -> 2
- net /wifi/C6_USB_DP: track 0.00 -> 13.0 mm, vias 0 -> 2
- net /power/CHG_DP: track 0.00 -> 11.0 mm, vias 0 -> 2
- net /power/USB_CC1: track 0.00 -> 10.5 mm, vias 0 -> 2
- net /mcu/P4_CSI_D0_P: track 0.00 -> 9.45 mm
- net /mcu/P4_CSI_D0_N: track 0.00 -> 9.45 mm
- net /mcu/P4_CSI_D1_N: track 0.00 -> 9.11 mm
- net /mcu/P4_CSI_D1_P: track 0.00 -> 9.11 mm
- net /mcu/P4_CSI_CK_N: track 0.00 -> 8.11 mm, vias 0 -> 2
- net /wifi/C6_USB_DN: track 0.00 -> 8.08 mm, vias 0 -> 2
- net /mcu/P4_CSI_CK_P: track 0.00 -> 7.90 mm, vias 0 -> 2
- net /lte/MDM_USB_DP: track 0.00 -> 7.14 mm, vias 0 -> 2
- net /mcu/P4_USB_DN: track 0.00 -> 7.02 mm, vias 0 -> 1
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- added copper zone on In2.Cu, net 3V3
- added copper zone on B.Cu, net GND
- added copper zone on F.Cu, net GND
- added copper zone on In2.Cu, net SYS
- added copper zone on In2.Cu, net VBAT_LTE

Commit message: Phase 5: SIM7600 RF feeds (MAIN/AUX/GNSS CPWG, pi-match inline, GND fence)
Co-Authored-By: Claude Opus 5.5 <noreply@anthropic.com>
Parts:
- moved R511 9.02 mm to (47.1, 31.4), turned to 0 degrees
- moved C522 6.95 mm to (49.5, 31.0)
- moved C521 6.57 mm to (45.6, 31.0), turned to 90 degrees
- moved C519 6.13 mm to (70.0, 42.8), turned to -90 degrees
- moved R509 1.36 mm to (71.5, 61.3)
- moved C517 1.29 mm to (70.0, 61.8), turned to -90 degrees
- moved L501 0.91 mm to (50.9, 31.4), turned to 180 degrees
- moved R510 0.85 mm to (71.5, 42.3), turned to 0 degrees
- moved C520 0.55 mm to (72.9, 42.8), turned to -90 degrees
- moved C518 0.21 mm to (72.9, 61.8), turned to -90 degrees
- moved J7 0.10 mm to (47.6, 29.8)
Routing:
- net /lte/ANT_MAIN: track 0.00 -> 5.30 mm
- net /lte/ANT_AUX: track 0.00 -> 5.30 mm
- net GND: track 0.00 -> 4.34 mm, vias 0 -> 8
- net /lte/RF_GNSS: track 0.00 -> 3.72 mm
- net /lte/ANT_GNSS: track 0.00 -> 3.18 mm
- net /lte/RF_MAIN: track 0.00 -> 2.50 mm
- net /lte/RF_AUX: track 0.00 -> 2.50 mm
